File: bluepill-protoboard/bluepill-protoboard.kicad_sch (KiCad schematic)
At the start: 35 parts, among them J1 Conn_01x20_Socket, J10 Conn_01x04_Pin, J11 Conn_01x04_Pin, J13 Conn_01x06_Pin, J14 Conn_01x04_Pin, J15 Conn_01x04_Pin, J2 Conn_01x17_Pin, J3 Conn_01x17_Pin, J4 Conn_01x17_Pin, J5 Conn_01x04_Pin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

Commit message: Update components
Parts:
- C1: value C -> 0.1
- C10, C8, C9: value C -> 47uF
- C11: value C -> 100nF
- C2: value C -> 0.47uF
- C3, C4: value C -> 22uF
- C5: value C -> 10pF
- C6: value C -> 1.5nF
- C7: value C -> 8.2nF
- D1: value D_Schottky_Filled -> 550mV
- L1: value L -> 22uH
- R1: value R -> 169K
- R2: value R -> 93.1K
- R3: value R -> 47.5K
- R4: value R -> 10.2K
- R5: value R -> 1.96K
Other:
- note added: "VIN 6V - 18V"
Changed lines of the file:
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@@
+    (effects (font (size 1.27 1.27)) (justify left bottom))
+  )
+  (text "VIN 6V - 18V" (at 17.78 116.84 0)
     (effects (font (size 1.27 1.27)) (justify left bottom))
   )
@@
       (effects (font (size 1.27 1.27)))
     )
-    (property "Value" "L" (at 147.32 116.84 90)
+    (property "Value" "22uH" (at 147.32 116.84 90)
       (effects (font (size 1.27 1.27)))
     )
@@
       (effects (font (size 1.27 1.27)) (justify left))
     )
-    (property "Value" "D_Schottky_Filled" (at 137.16 124.1425 90)
+    (property "Value" "550mV" (at 137.16 124.1425 90)
       (effects (font (size 1.27 1.27)) (justify left))
     )
@@
       (effects (font (size 1.27 1.27)) (justify left))
     )
-    (property "Value" "C" (at 74.93 146.05 0)
+    (property "Value" "10pF" (at 74.93 146.05 0)
       (effects (font (size 1.27 1.27)) (justify left))
     )
@@
       (effects (font (size 1.27 1.27)) (justify left))
     )
-    (property "Value" "C" (at 36.83 180.34 0)
+    (property "Value" "0.1" (at 36.83 180.34 0)
       (effects (font (size 1.27 1.27)) (justify left))
     )
@@
       (effects (font (size 1.27 1.27)) (justify left))
     )
-    (property "Value" "C" (at 67.31 180.34 0)
+    (property "Value" "0.47uF" (at 67.31 180.34 0)
       (effects (font (size 1.27 1.27)) (justify left))
     )
@@
       (effects (font (size 1.27 1.27)) (justify left))
     )
-    (property "Value" "C" (at 45.72 128.27 0)
+    (property "Value" "22uF" (at 45.72 128.27 0)
       (effects (font (size 1.27 1.27)) (justify left))
     )
@@
       (effects (font (size 1.27 1.27)) (justify left))
     )
-    (property "Value" "C" (at 129.54 116.84 0)
+    (property "Value" "100nF" (at 129.54 116.84 0)
       (effects (font (size 1.27 1.27)) (justify left))
     )
@@
       (effects (font (size 1.27 1.27)) (justify left))
     )
-    (property "Value" "R" (at 66.04 134.62 0)
+    (property "Value" "93.1K" (at 66.04 134.62 0)
       (effects (font (size 1.27 1.27)) (justify left))
     )
@@
       (effects (font (size 1.27 1.27)) (justify left))
     )
-    (property "Value" "R" (at 160.02 146.05 0)
+    (property "Value" "1.96K" (at 160.02 146.05 0)
       (effects (font (size 1.27 1.27)) (justify left))
     )
@@
       (effects (font (size 1.27 1.27)) (justify left))
     )
-    (property "Value" "C" (at 55.88 128.27 0)
+    (property "Value" "22uF" (at 55.88 128.27 0)
       (effects (font (size 1.27 1.27)) (justify left))
     )
@@
       (effects (font (size 1.27 1.27)) (justify left))
     )
-    (property "Value" "R" (at 160.02 129.54 0)
+    (property "Value" "10.2K" (at 160.02 129.54 0)
       (effects (font (size 1.27 1.27)) (justify left))
     )
@@
       (effects (font (size 1.27 1.27)) (justify left))
     )
-    (property "Value" "R" (at 83.82 134.62 0)
+    (property "Value" "47.5K" (at 83.82 134.62 0)
       (effects (font (size 1.27 1.27)) (justify left))
     )
@@
       (effects (font (size 1.27 1.27)) (justify left))
     )
-    (property "Value" "C" (at 85.09 146.05 0)
+    (property "Value" "1.5nF" (at 85.09 146.05 0)
       (effects (font (size 1.27 1.27)) (justify left))
     )
@@
       (effects (font (size 1.27 1.27)) (justify left))
     )
-    (property "Value" "C" (at 194.31 130.81 0)
+    (property "Value" "47uF" (at 194.31 130.81 0)
       (effects (font (size 1.27 1.27)) (justify left))
     )
@@
       (effects (font (size 1.27 1.27)) (justify left))
     )
-    (property "Value" "C" (at 95.25 146.05 0)
+    (property "Value" "8.2nF" (at 95.25 146.05 0)
       (effects (font (size 1.27 1.27)) (justify left))
     )
@@
       (effects (font (size 1.27 1.27)) (justify left))
     )
-    (property "Value" "R" (at 66.04 121.92 0)
+    (property "Value" "169K" (at 66.04 121.92 0)
       (effects (font (size 1.27 1.27)) (justify left))
     )
@@
       (effects (font (size 1.27 1.27)) (justify left))
     )
-    (property "Value" "C" (at 173.99 130.81 0)
+    (property "Value" "47uF" (at 173.99 130.81 0)
       (effects (font (size 1.27 1.27)) (justify left))
     )
@@
       (effects (font (size 1.27 1.27)) (justify left))
     )
-    (property "Value" "C" (at 184.15 130.81 0)
-      (effects (font (size 1.27 1.27)) (justify left))
-    )
+    (property "Value" "47uF" (at 184.15 130.81 0)
+      (effects (font (size 1.27 1.27)) (justify left))
+    )

Commit message: Start PCB
Parts:
- C1, C10, C11, C2, C3, C4, C5, C6, C7, C8, C9: footprint (none) -> Capacitor_SMD:C_0402_1005Metric
- D1: footprint (none) -> Diode_SMD:D_01005_0402Metric
- J1, J8: footprint (none) -> Connector_PinSocket_2.54mm:PinSocket_1x20_P2.54mm_Vertical
- J10, J11, J14, J15, J5: footprint (none) -> Connector_PinHeader_2.54mm:PinHeader_1x04_P2.54mm_Vertical
- J13: footprint (none) -> Connector_PinHeader_2.54mm:PinHeader_1x06_P2.54mm_Vertical
- J2, J3, J4: value Conn_01x17_Pin -> Conn_01x16_Pin; footprint (none) -> Connector_PinHeader_2.54mm:PinHeader_1x16_P2.54mm_Vertical
- J50: footprint (none) -> Connector_BarrelJack:BarrelJack_Horizontal
- J6, J7, J9: footprint (none) -> Connector_PinHeader_2.54mm:PinHeader_1x17_P2.54mm_Vertical
- L1: footprint (none) -> Inductor_SMD:L_0402_1005Metric
- R1, R2, R3, R4, R5: footprint (none) -> Resistor_SMD:R_0402_1005Metric
Changed lines of the file:
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@@
       (effects (font (size 1.27 1.27)))
     )
-    (property "Footprint" "" (at 147.32 119.38 0)
+    (property "Footprint" "Inductor_SMD:L_0402_1005Metric" (at 147.32 119.38 0)
       (effects (font (size 1.27 1.27)) hide)
     )
@@
       (effects (font (size 1.27 1.27)))
     )
-    (property "Footprint" "" (at 26.67 120.904 0)
+    (property "Footprint" "Connector_BarrelJack:BarrelJack_Horizontal" (at 26.67 120.904 0)
       (effects (font (size 1.27 1.27)) hide)
     )
@@
       (effects (font (size 1.27 1.27)) (justify left))
     )
-    (property "Footprint" "" (at 134.62 123.19 0)
+    (property "Footprint" "Diode_SMD:D_01005_0402Metric" (at 134.62 123.19 0)
       (effects (font (size 1.27 1.27)) hide)
     )
@@
       (effects (font (size 1.27 1.27)) (justify left))
     )
-    (property "Footprint" "" (at 72.0852 148.59 0)
+    (property "Footprint" "Capacitor_SMD:C_0402_1005Metric" (at 72.0852 148.59 0)
       (effects (font (size 1.27 1.27)) hide)
     )
@@
       (effects (font (size 1.27 1.27)) (justify left))
     )
-    (property "Footprint" "" (at 33.9852 182.88 0)
+    (property "Footprint" "Capacitor_SMD:C_0402_1005Metric" (at 33.9852 182.88 0)
       (effects (font (size 1.27 1.27)) hide)
     )
@@
       (effects (font (size 1.27 1.27)))
     )
-    (property "Footprint" "" (at 248.92 57.15 0)
+    (property "Footprint" "Connector_PinHeader_2.54mm:PinHeader_1x17_P2.54mm_Vertical" (at 248.92 57.15 0)
       (effects (font (size 1.27 1.27)) hide)
     )
@@
       (effects (font (size 1.27 1.27)))
     )
-    (property "Value" "Conn_01x17_Pin" (at 46.99 73.66 0)
-      (effects (font (size 1.27 1.27)))
-    )
-    (property "Footprint" "" (at 44.45 48.26 0)
+    (property "Value" "Conn_01x16_Pin" (at 46.99 73.66 0)
+      (effects (font (size 1.27 1.27)))
+    )
+    (property "Footprint" "Connector_PinHeader_2.54mm:PinHeader_1x16_P2.54mm_Vertical" (at 44.45 48.26 0)
       (effects (font (size 1.27 1.27)) hide)
     )
@@
       (effects (font (size 1.27 1.27)) (justify left))
     )
-    (property "Footprint" "" (at 64.4652 182.88 0)
+    (property "Footprint" "Capacitor_SMD:C_0402_1005Metric" (at 64.4652 182.88 0)
       (effects (font (size 1.27 1.27)) hide)
     )
@@
       (effects (font (size 1.27 1.27)) (justify left))
     )
-    (property "Footprint" "" (at 42.8752 130.81 0)
+    (property "Footprint" "Capacitor_SMD:C_0402_1005Metric" (at 42.8752 130.81 0)
       (effects (font (size 1.27 1.27)) hide)
     )
@@
       (effects (font (size 1.27 1.27)))
     )
-    (property "Footprint" "" (at 257.81 130.81 0)
+    (property "Footprint" "Connector_PinHeader_2.54mm:PinHeader_1x04_P2.54mm_Vertical" (at 257.81 130.81 0)
       (effects (font (size 1.27 1.27)) hide)
     )
@@
       (effects (font (size 1.27 1.27)))
     )
-    (property "Value" "Conn_01x17_Pin" (at 113.03 26.67 0)
-      (effects (font (size 1.27 1.27)))
-    )
-    (property "Footprint" "" (at 110.49 48.26 0)
+    (property "Value" "Conn_01x16_Pin" (at 113.03 26.67 0)
+      (effects (font (size 1.27 1.27)))
+    )
+    (property "Footprint" "Connector_PinHeader_2.54mm:PinHeader_1x16_P2.54mm_Vertical" (at 110.49 48.26 0)
       (effects (font (size 1.27 1.27)) hide)
     )
@@
       (effects (font (size 1.27 1.27)) (justify left))
     )
-    (property "Footprint" "" (at 126.6952 119.38 0)
+    (property "Footprint" "Capacitor_SMD:C_0402_1005Metric" (at 126.6952 119.38 0)
       (effects (font (size 1.27 1.27)) hide)
     )
@@
       (effects (font (size 1.27 1.27)))
     )
-    (property "Footprint" "" (at 200.66 40.64 0)
+    (property "Footprint" "Connector_PinHeader_2.54mm:PinHeader_1x04_P2.54mm_Vertical" (at 200.66 40.64 0)
       (effects (font (size 1.27 1.27)) hide)
     )
@@
       (effects (font (size 1.27 1.27)) (justify left))
     )
-    (property "Footprint" "" (at 61.722 133.35 90)
+    (property "Footprint" "Resistor_SMD:R_0402_1005Metric" (at 61.722 133.35 90)
       (effects (font (size 1.27 1.27)) hide)
     )
@@
       (effects (font (size 1.27 1.27)) (justify left))
     )
-    (property "Footprint" "" (at 155.702 144.78 90)
+    (property "Footprint" "Resistor_SMD:R_0402_1005Metric" (at 155.702 144.78 90)
       (effects (font (size 1.27 1.27)) hide)
     )
@@
       (effects (font (size 1.27 1.27)))
     )
-    (property "Footprint" "" (at 231.14 57.15 0)
+    (property "Footprint" "Connector_PinHeader_2.54mm:PinHeader_1x17_P2.54mm_Vertical" (at 231.14 57.15 0)
       (effects (font (size 1.27 1.27)) hide)
     )
@@
       (effects (font (size 1.27 1.27)) (justify left))
     )
-    (property "Footprint" "" (at 53.0352 130.81 0)
+    (property "Footprint" "Capacitor_SMD:C_0402_1005Metric" (at 53.0352 130.81 0)
       (effects (font (size 1.27 1.27)) hide)
     )
@@
       (effects (font (size 1.27 1.27)) (justify left))
     )
-    (property "Footprint" "" (at 156.21 50.8 0)
+    (property "Footprint" "Connector_PinSocket_2.54mm:PinSocket_1x20_P2.54mm_Vertical" (at 156.21 50.8 0)
       (effects (font (size 1.27 1.27)) hide)
     )
@@
       (effects (font (size 1.27 1.27)) (justify left))
     )
-    (property "Footprint" "" (at 155.702 128.27 90)
+    (property "Footprint" "Resistor_SMD:R_0402_1005Metric" (at 155.702 128.27 90)
       (effects (font (size 1.27 1.27)) hide)
     )
@@
       (effects (font (size 1.27 1.27)) (justify left))
     )
-    (property "Footprint" "" (at 79.502 133.35 90)
+    (property "Footprint" "Resistor_SMD:R_0402_1005Metric" (at 79.502 133.35 90)
       (effects (font (size 1.27 1.27)) hide)
     )
@@
       (effects (font (size 1.27 1.27)) (justify left))
     )
-    (property "Footprint" "" (at 82.2452 148.59 0)
+    (property "Footprint" "Capacitor_SMD:C_0402_1005Metric" (at 82.2452 148.59 0)
       (effects (font (size 1.27 1.27)) hide)
     )
@@
       (effects (font (size 1.27 1.27)) (justify left))
     )
-    (property "Footprint" "" (at 191.4652 133.35 0)
+    (property "Footprint" "Capacitor_SMD:C_0402_1005Metric" (at 191.4652 133.35 0)
       (effects (font (size 1.27 1.27)) hide)
     )
@@
       (effects (font (size 1.27 1.27)) (justify left))
     )
-    (property "Footprint" "" (at 92.4052 148.59 0)
+    (property "Footprint" "Capacitor_SMD:C_0402_1005Metric" (at 92.4052 148.59 0)
       (effects (font (size 1.27 1.27)) hide)
     )
@@
       (effects (font (size 1.27 1.27)) (justify left))
     )
-    (property "Footprint" "" (at 61.722 120.65 90)
+    (property "Footprint" "Resistor_SMD:R_0402_1005Metric" (at 61.722 120.65 90)
       (effects (font (size 1.27 1.27)) hide)
     )
@@
       (effects (font (size 1.27 1.27)))
     )
-    (property "Footprint" "" (at 222.25 130.81 0)
+    (property "Footprint" "Connector_PinHeader_2.54mm:PinHeader_1x04_P2.54mm_Vertical" (at 222.25 130.81 0)
       (effects (font (size 1.27 1.27)) hide)
     )
@@
       (effects (font (size 1.27 1.27)))
     )
-    (property "Footprint" "" (at 147.32 87.63 0)
+    (property "Footprint" "Connector_PinHeader_2.54mm:PinHeader_1x06_P2.54mm_Vertical" (at 147.32 87.63 0)
       (effects (font (size 1.27 1.27)) hide)
     )
@@
       (effects (font (size 1.27 1.27)))
     )
-    (property "Footprint" "" (at 179.07 55.88 0)
+    (property "Footprint" "Connector_PinHeader_2.54mm:PinHeader_1x17_P2.54mm_Vertical" (at 179.07 55.88 0)
       (effects (font (size 1.27 1.27)) hide)
     )
@@
       (effects (font (size 1.27 1.27)))
     )
-    (property "Value" "Conn_01x17_Pin" (at 29.21 26.67 0)
-      (effects (font (size 1.27 1.27)))
-    )
-    (property "Footprint" "" (at 26.67 48.26 0)
+    (property "Value" "Conn_01x16_Pin" (at 29.21 26.67 0)
+      (effects (font (size 1.27 1.27)))
+    )
+    (property "Footprint" "Connector_PinHeader_2.54mm:PinHeader_1x16_P2.54mm_Vertical" (at 26.67 48.26 0)
       (effects (font (size 1.27 1.27)) hide)
     )
@@
       (effects (font (size 1.27 1.27)))
     )
-    (property "Footprint" "" (at 240.03 130.81 0)
+    (property "Footprint" "Connector_PinHeader_2.54mm:PinHeader_1x04_P2.54mm_Vertical" (at 240.03 130.81 0)
       (effects (font (size 1.27 1.27)) hide)
     )
@@
       (effects (font (size 1.27 1.27)) (justify left))
     )
-    (property "Footprint" "" (at 171.1452 133.35 0)
+    (property "Footprint" "Capacitor_SMD:C_0402_1005Metric" (at 171.1452 133.35 0)
       (effects (font (size 1.27 1.27)) hide)
     )
@@
       (effects (font (size 1.27 1.27)) (justify left))
     )
-    (property "Footprint" "" (at 133.35 50.8 0)
+    (property "Footprint" "Connector_PinSocket_2.54mm:PinSocket_1x20_P2.54mm_Vertical" (at 133.35 50.8 0)
       (effects (font (size 1.27 1.27)) hide)
     )
@@
       (effects (font (size 1.27 1.27)) (justify left))
     )
-    (property "Footprint" "" (at 181.3052 133.35 0)
+    (property "Footprint" "Capacitor_SMD:C_0402_1005Metric" (at 181.3052 133.35 0)
       (effects (font (size 1.27 1.27)) hide)
     )
@@
       (effects (font (size 1.27 1.27)))
     )
-    (property "Footprint" "" (at 82.55 66.04 0)
-      (effects (font (size 1.27 1.27)) hide)
-    )
+    (property "Footprint" "Connector_PinHeader_2.54mm:PinHeader_1x04_P2.54mm_Vertical" (at 82.55 66.04 0)
+      (effects (font (size 1.27 1.27)) hide)
+    )
