File: bluepill-protoboard/bluepill-protoboard.kicad_pcb (KiCad board)
At the start: 2 copper layers, 35 parts, among them J1 Conn_01x20_Socket, J10 Conn_01x04_Pin, J11 Conn_01x04_Pin, J13 Conn_01x06_Pin, J14 Conn_01x04_Pin, J15 Conn_01x04_Pin, J2 Conn_01x16_Pin, J3 Conn_01x16_Pin, J4 Conn_01x16_Pin, J5 Conn_01x04_Pin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

Commit message: More PCB
Parts:
- moved J50 177.4 mm to (77.1, 116.8)
- moved J15 119.1 mm to (139.7, 68.6), turned to -90 degrees
- moved J14 113.6 mm to (139.7, 73.7), turned to -90 degrees
- moved J11 112.0 mm to (139.7, 61.0), turned to -90 degrees
- moved J10 102.4 mm to (139.7, 94.0), turned to -90 degrees
- moved J5 99.0 mm to (139.7, 78.7), turned to -90 degrees
